Commit message: corrections and test done, remember : can not be used in .urdf comment

File: urdf/barista_robot_model.urdf (robot description, URDF)
Before this commit: robot barista, 9 links, 8 joints
Joints:
- joint right_wheel_joint: origin xyz=0 -0.150 -0.0775 rpy=0 0 0 -> xyz=0 +0.150 -0.0775 rpy=0 0 0
- joint standoff_rod_xnyn_joint: origin xyz=-0.150 -0.150 0.1875 rpy=0 0 0 -> xyz=-0.075 -0.075 0.1875 rpy=0 0 0
- joint standoff_rod_xnyp_joint: origin xyz=-0.150 0.150 0.1875 rpy=0 0 0 -> xyz=-0.075 0.075 0.1875 rpy=0 0 0
- joint standoff_rod_xpyn_joint: origin xyz=0.150 -0.150 0.1875 rpy=0 0 0 -> xyz=0.075 -0.075 0.1875 rpy=0 0 0
- joint standoff_rod_xpyp_joint: origin xyz=0.150 0.150 0.1875 rpy=0 0 0 -> xyz=0.075 0.075 0.1875 rpy=0 0 0

Commit message: caster wheels placed correctly

File: urdf/barista_robot_model.urdf (robot description, URDF)
Before this commit: robot barista, 9 links, 8 joints
Links:
- added link back_caster_wheel_p; collision cylinder length=0.002 radius=0.010; visual cylinder length=0.002 radius=0.010
- added link back_caster_wheel_r; collision cylinder length=0.002 radius=0.010; visual cylinder length=0.002 radius=0.010
- added link back_caster_wheel_y; collision sphere radius=0.0352; visual sphere radius=0.0352
- added link front_caster_wheel_p; collision cylinder length=0.002 radius=0.010; visual cylinder length=0.002 radius=0.010
- added link front_caster_wheel_r; collision cylinder length=0.002 radius=0.010; visual cylinder length=0.002 radius=0.010
- added link front_caster_wheel_y; collision sphere radius=0.0352; visual sphere radius=0.0352
Joints:
- added joint back_pitch_joint: type continuous, parent back_caster_wheel_r, child back_caster_wheel_p, origin xyz=0 0 0 rpy=0 0 0, axis 0 1 0, limit effort=1000.0 velocity=100.0
- added joint back_roll_joint: type continuous, parent chassis, child back_caster_wheel_r, origin xyz=-0.100 0 -0.0775 rpy=0 0 0, axis 1 0 0, limit effort=1000.0 velocity=100.0
- added joint back_yaw_joint: type continuous, parent back_caster_wheel_p, child back_caster_wheel_y, origin xyz=0 0 0 rpy=0 0 0, axis 0 0 1, limit effort=1000.0 velocity=100.0
- added joint front_pitch_joint: type continuous, parent front_caster_wheel_r, child front_caster_wheel_p, origin xyz=0 0 0 rpy=0 0 0, axis 0 1 0, limit effort=1000.0 velocity=100.0
- added joint front_roll_joint: type continuous, parent chassis, child front_caster_wheel_r, origin xyz=0.100 0 -0.0775 rpy=0 0 0, axis 1 0 0, limit effort=1000.0 velocity=100.0
- added joint front_yaw_joint: type continuous, parent front_caster_wheel_p, child front_caster_wheel_y, origin xyz=0 0 0 rpy=0 0 0, axis 0 0 1, limit effort=1000.0 velocity=100.0

Commit message: laser model was added and gazebo stuff

File: urdf/barista_robot_model.urdf (robot description, URDF)
Before this commit: robot barista, 15 links, 14 joints
Links:
- added link laser_model; collision mesh filename=package://barista_robot_description/meshes/hokuyo_urg_04lx.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; visual mesh filename=package://barista_robot_description/meshes/hokuyo_urg_04lx.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
Joints:
- added joint laser_model_link_joint: type fixed, parent chassis, child laser_model, origin xyz=0.120 0.0 0.0775 rpy=0 0 0

Commit message: inertias calculated

File: urdf/barista_robot_model.urdf (robot description, URDF)
Before this commit: robot barista, 16 links, 15 joints
Links:
- link back_caster_wheel_p: mass None -> 0.01
- link back_caster_wheel_r: mass None -> 0.01
- link back_caster_wheel_y: mass None -> 0.5
- link chassis: mass None -> 10.0
- link cup_holder_tray: mass None -> 5.0
- link front_caster_wheel_p: mass None -> 0.01
- link front_caster_wheel_r: mass None -> 0.01
- link front_caster_wheel_y: mass None -> 0.5
- link laser_model: mass None -> 0.16
- link left_wheel: mass None -> 0.5
- link right_wheel: mass None -> 0.5
- link standoff_rod_xnyn: mass None -> 0.2
- link standoff_rod_xnyp: mass None -> 0.2
- link standoff_rod_xpyn: mass None -> 0.2
- link standoff_rod_xpyp: mass None -> 0.2

Commit message: some changes made, but the robot launches incomplete

File: urdf/barista_robot_model.urdf (robot description, URDF)
Before this commit: robot barista, 16 links, 15 joints
Links:
- link back_caster_wheel_y: geometry collision sphere radius=0.0176; visual sphere radius=0.0176
- link front_caster_wheel_y: geometry collision sphere radius=0.0176; visual sphere radius=0.0176
Joints:
- joint back_roll_joint: origin xyz=-0.100 0 -0.0775 rpy=0 0 0 -> xyz=-0.100 0 -0.0951 rpy=0 0 0
- joint front_roll_joint: origin xyz=0.100 0 -0.0775 rpy=0 0 0 -> xyz=0.100 0 -0.0951 rpy=0 0 0

Commit message: 3 launches generated to test the robot's deploy

File: urdf/barista_robot_model.urdf (robot description, URDF)
Before this commit: robot barista, 16 links, 15 joints
Joints:
- joint left_wheel_joint: origin xyz=0 -0.150 -0.0775 rpy=0 0 0 -> xyz=0 +0.150 -0.0775 rpy=0 0 0
- joint right_wheel_joint: origin xyz=0 +0.150 -0.0775 rpy=0 0 0 -> xyz=0 -0.150 -0.0775 rpy=0 0 0

Commit message: 1 launch is ready and was improved the laser pos

File: urdf/barista_robot_model.urdf (robot description, URDF)
Before this commit: robot barista, 16 links, 15 joints
Joints:
- joint laser_model_link_joint: origin xyz=0.120 0.0 0.0775 rpy=0 0 0 -> xyz=0.120 0.0 +0.1275 rpy=0 0 0

Commit message: the diameter of the rods were corrected

File: urdf/barista_robot_model.urdf (robot description, URDF)
Before this commit: robot barista, 16 links, 15 joints
Links:
- link standoff_rod_xnyn: geometry collision cylinder length=0.220 radius=0.010; visual cylinder length=0.220 radius=0.010
- link standoff_rod_xnyp: geometry collision cylinder length=0.220 radius=0.010; visual cylinder length=0.220 radius=0.010
- link standoff_rod_xpyn: geometry collision cylinder length=0.220 radius=0.010; visual cylinder length=0.220 radius=0.010
- link standoff_rod_xpyp: geometry collision cylinder length=0.220 radius=0.010; visual cylinder length=0.220 radius=0.010
