Commit message: corrections done to every xacro file - xacro robot is working well

File: xacro/barista_robot_model.urdf.xacro (robot description, xacro)
@@ -2,5 +2,5 @@
 <robot xmlns:xacro="http://www.ros.org/wiki/xacro" name="barista">
 <xacro:property name="robot_name" value="$(arg robot_name)"/>
-<xacro:property name="include_laser" value="$(arg include_laser, True)"/>
+<xacro:property name="include_laser" value="$(arg include_laser)"/>
 <!--include the macros-->
 <xacro:include filename="$(find barista_robot_description)/xacro/wheel.xacro"/>
@@ -33,7 +33,9 @@
 <xacro:property name="wheel_separation" value="0.300"/>
 <!--caster parameters-->
-<xacro:property name="caster_radius" value="0.0352"/>
+<xacro:property name="caster_radius" value="0.020"/>
 <xacro:property name="caster_mass" value="0.1"/>
 <xacro:property name="caster_material" value="blue"/>
+<!--laser parameters-->
+<xacro:property name="laser_mass" value="0.160"/>
 <!--material alpha-->
 <xacro:property name="alpha" value="0.7"/>
@@ -55,6 +57,6 @@
 <link name="base_link"/>
 <!--generate the chassis and cup holder tray-->
-<xacro::cup_holder_tray name="chassis" radius="${chassis_diameter/2}" height="${chassis_height}" mass="${chassis_mass}" material="${chassis_material}"/>
-<xacro::cup_holder_tray name="cup_holder_tray" radius="${tray_diameter/2}" height="${tray_height}" mass="${tray_mass}" material="${tray_material}"/>
+<xacro:cup_holder_tray name="chassis" radius="${chassis_diameter/2}" height="${chassis_height}" mass="${chassis_mass}" material="${chassis_material}"/>
+<xacro:cup_holder_tray name="cup_holder_tray" radius="${tray_diameter/2}" height="${tray_height}" mass="${tray_mass}" material="${tray_material}"/>
 <!--generate 4 standoff rods-->
 <xacro:standoff name="xpyp_standoff" radius="${standoff_diameter/2}" height="${standoff_height}" mass="${standoff_mass}" material="${standoff_material}"/>
@@ -70,5 +72,5 @@
 <!--generate the laser scanner-->
 <xacro:if value="${include_laser}">
-    <xacro:laser_scanner name="laser_scanner" radius="${tray_diameter/2}" height="${tray_height}" mass="${tray_mass}" material="${tray_material}"/>
+    <xacro:laser_scanner name="laser_scanner" mass="${laser_mass}"/>
 </xacro:if>
 <!--define the robot joints-->
@@ -126,6 +128,6 @@
 <joint name="front_caster_joint" type="continuous">
     <parent link="chassis"/>
-    <child link="front_caster"/>
-    <origin xyz="${chassis_diameter/3} 0 ${-chassis_height/2-caster_radius}" rpy="0 0 0"/>
+    <child link="front_caster_wheel_r"/>
+    <origin xyz="${chassis_diameter/3} 0 ${-chassis_height/2-wheel_diameter/2+caster_radius}" rpy="0 0 0"/>
     <axis xyz="1 0 0" rpy="0 0 0"/>
     <limit effort="1000.0" velocity="100.0" />
@@ -134,6 +136,6 @@
 <joint name="back_caster_joint" type="continuous">
     <parent link="chassis"/>
-    <child link="back_caster"/>
-    <origin xyz="${-chassis_diameter/3} 0 ${-chassis_height/2-caster_radius}" rpy="0 0 0"/>
+    <child link="back_caster_wheel_r"/>
+    <origin xyz="${-chassis_diameter/3} 0 ${-chassis_height/2-wheel_diameter/2+caster_radius}" rpy="0 0 0"/>
     <axis xyz="1 0 0" rpy="0 0 0"/>
     <limit effort="1000.0" velocity="100.0" />
@@ -153,4 +155,5 @@
     <plugin name="joint_state_publisher_node" filename="libgazebo_ros_joint_state_publisher.so">
         <ros>
+            <namespace>/${robot_name}</namespace>
             <remapping>~/out:=joint_states</remapping>
         </ros>
@@ -169,4 +172,8 @@
 <gazebo>
     <plugin filename="libgazebo_ros_diff_drive.so" name="differential_drive_controller_node">
+        <ros>
+            <namespace>/${robot_name}</namespace>
+            <remapping>/out:=cmd_vel</remapping>
+        </ros>
         <!-- wheels -->
         <left_joint>left_wheel_joint</left_joint>
@@ -232,6 +239,8 @@
     <material>Gazebo/White</material>
 </gazebo>
-<gazebo reference="laserscanner">
-    <material>Gazebo/DarkGrey</material>
-</gazebo>
+<xacro:if value="${include_laser}">
+    <gazebo reference="laser_scanner">
+        <material>Gazebo/DarkGrey</material>
+    </gazebo>
+</xacro:if>
 </robot>

File: xacro/cup_holder_tray.xacro (robot description, xacro)
@@ -1,5 +1,5 @@
 <?xml version="1.0"?>
 <robot xmlns:xacro="http://www.ros.org/wiki/xacro">
-<xacro:macro name="cup_holder_tray" params="name, radius, height, mass, material">
+<xacro:macro name="cup_holder_tray" params="name radius height mass material">
     <link name="${name}">
         <visual>

File: xacro/laser_scanner.xacro (robot description, xacro)
@@ -1,5 +1,5 @@
 <?xml version="1.0"?>
 <robot xmlns:xacro="http://www.ros.org/wiki/xacro">
-<xacro:macro name="laser_scanner" params="name, mass">
+<xacro:macro name="laser_scanner" params="name mass">
     <!--the origin is 0.05 over the base-->
     <xacro:property name="laser_r" value="0.05"/>

File: xacro/standoff.xacro (robot description, xacro)
@@ -1,5 +1,5 @@
 <?xml version="1.0"?>
 <robot xmlns:xacro="http://www.ros.org/wiki/xacro">
-<xacro:macro name="standoff" params="name, radius, height, mass, material">
+<xacro:macro name="standoff" params="name radius height mass material">
     <link name="${name}">
         <visual>

File: xacro/wheel.xacro (robot description, xacro)
@@ -1,5 +1,5 @@
 <?xml version="1.0"?>
 <robot xmlns:xacro="http://www.ros.org/wiki/xacro">
-<xacro:macro name="wheel" params="name, radius, width, mass, material">
+<xacro:macro name="wheel" params="name radius width mass material">
     <link name="${name}">
         <visual>
@@ -25,9 +25,9 @@
     </link>
 </xacro:macro>
-<xacro:macro name="caster" params="name, radius, mass, material">
+<xacro:macro name="caster" params="name radius mass material">
   <!--local variables-->
-  <xacro:let name="cylinder_r" value="${radius/3}"/>
-  <xacro:let name="cylinder_w" value="${radius/15}"/>
-  <xacro:let name="cylinder_m" value="${mass/5}"/>
+  <xacro:property name="cylinder_r" value="${radius/3}"/>
+  <xacro:property name="cylinder_h" value="${radius/15}"/>
+  <xacro:property name="cylinder_m" value="${mass/5}"/>
   <link name="${name}_wheel_r">
     <visual>

Commit message: improves were done. now is easy to instantiate multiple robots

File: xacro/barista_robot_model.urdf.xacro (robot description, xacro)
@@ -3,4 +3,5 @@
 <xacro:property name="robot_name" value="$(arg robot_name)"/>
 <xacro:property name="include_laser" value="$(arg include_laser)"/>
+<xacro:property name="robot_color" value="$(arg robot_color)"/>
 <!--include the macros-->
 <xacro:include filename="$(find barista_robot_description)/xacro/wheel.xacro"/>
@@ -222,8 +223,8 @@
 </gazebo>
 <gazebo reference="chassis">
-    <material>Gazebo/Red</material>
+    <material>${robot_color}</material>
 </gazebo>
 <gazebo reference="cup_holder_tray">
-    <material>Gazebo/Red</material>
+    <material>${robot_color}</material>
 </gazebo>
 <gazebo reference="xpyp_standoff">

File: xacro/laser_scanner.xacro (robot description, xacro)
@@ -33,6 +33,6 @@
           <scan>
             <horizontal>
-              <samples>200</samples>
-              <resolution>1.0</resolution>
+              <samples>360</samples>
+              <!--resolution>1.0</resolution-->
               <min_angle>-3.14</min_angle>
               <max_angle>3.14</max_angle>
@@ -46,7 +46,8 @@
         <always_on>true</always_on>
         <visualize>true</visualize>
-        <update_rate>100.0</update_rate>
+        <update_rate>20.0</update_rate>
         <plugin name="laser_scanner_node" filename="libgazebo_ros_ray_sensor.so">
           <ros>
+            <namespace>/${robot_name}</namespace>
             <remapping>~/out:=scan</remapping>
           </ros>

Commit message: simulation of multiple robots done

File: xacro/barista_robot_model.urdf.xacro (robot description, xacro)
@@ -56,61 +56,61 @@
 <!--define the robot body-->
 <!--base link-->
-<link name="base_link"/>
+<link name="${robot_name}/base_link"/>
 <!--generate the chassis and cup holder tray-->
-<xacro:cup_holder_tray name="chassis" radius="${chassis_diameter/2}" height="${chassis_height}" mass="${chassis_mass}" material="${chassis_material}"/>
-<xacro:cup_holder_tray name="cup_holder_tray" radius="${tray_diameter/2}" height="${tray_height}" mass="${tray_mass}" material="${tray_material}"/>
+<xacro:cup_holder_tray name="${robot_name}/chassis" radius="${chassis_diameter/2}" height="${chassis_height}" mass="${chassis_mass}" material="${chassis_material}"/>
+<xacro:cup_holder_tray name="${robot_name}/cup_holder_tray" radius="${tray_diameter/2}" height="${tray_height}" mass="${tray_mass}" material="${tray_material}"/>
 <!--generate 4 standoff rods-->
-<xacro:standoff name="xpyp_standoff" radius="${standoff_diameter/2}" height="${standoff_height}" mass="${standoff_mass}" material="${standoff_material}"/>
-<xacro:standoff name="xpyn_standoff" radius="${standoff_diameter/2}" height="${standoff_height}" mass="${standoff_mass}" material="${standoff_material}"/>
-<xacro:standoff name="xnyp_standoff" radius="${standoff_diameter/2}" height="${standoff_height}" mass="${standoff_mass}" material="${standoff_material}"/>
-<xacro:standoff name="xnyn_standoff" radius="${standoff_diameter/2}" height="${standoff_height}" mass="${standoff_mass}" material="${standoff_material}"/>
+<xacro:standoff name="${robot_name}/xpyp_standoff" radius="${standoff_diameter/2}" height="${standoff_height}" mass="${standoff_mass}" material="${standoff_material}"/>
+<xacro:standoff name="${robot_name}/xpyn_standoff" radius="${standoff_diameter/2}" height="${standoff_height}" mass="${standoff_mass}" material="${standoff_material}"/>
+<xacro:standoff name="${robot_name}/xnyp_standoff" radius="${standoff_diameter/2}" height="${standoff_height}" mass="${standoff_mass}" material="${standoff_material}"/>
+<xacro:standoff name="${robot_name}/xnyn_standoff" radius="${standoff_diameter/2}" height="${standoff_height}" mass="${standoff_mass}" material="${standoff_material}"/>
 <!--generate 2 wheels-->
-<xacro:wheel name="left_wheel" radius="${wheel_diameter/2}" width="${wheel_width}" mass="${wheel_mass}" material="${wheel_material}"/>
-<xacro:wheel name="right_wheel" radius="${wheel_diameter/2}" width="${wheel_width}" mass="${wheel_mass}" material="${wheel_material}"/>
+<xacro:wheel name="${robot_name}/left_wheel" radius="${wheel_diameter/2}" width="${wheel_width}" mass="${wheel_mass}" material="${wheel_material}"/>
+<xacro:wheel name="${robot_name}/right_wheel" radius="${wheel_diameter/2}" width="${wheel_width}" mass="${wheel_mass}" material="${wheel_material}"/>
 <!--generate 2 caster wheels-->
-<xacro:caster name="front_caster" radius="${caster_radius}" mass="${caster_mass}" material="${caster_material}"/>
-<xacro:caster name="back_caster" radius="${caster_radius}" mass="${caster_mass}" material="${caster_material}"/>
+<xacro:caster name="${robot_name}/front_caster" radius="${caster_radius}" mass="${caster_mass}" material="${caster_material}"/>
+<xacro:caster name="${robot_name}/back_caster" radius="${caster_radius}" mass="${caster_mass}" material="${caster_material}"/>
 <!--generate the laser scanner-->
 <xacro:if value="${include_laser}">
-    <xacro:laser_scanner name="laser_scanner" mass="${laser_mass}"/>
+    <xacro:laser_scanner name="${robot_name}/laser_scanner" mass="${laser_mass}"/>
 </xacro:if>
 <!--define the robot joints-->
 <!--base_link and chassis-->
 <joint name="base_link_joint" type="fixed">
-    <parent link="base_link"/>
-    <child link="chassis"/>
+    <parent link="${robot_name}/base_link"/>
+    <child link="${robot_name}/chassis"/>
     <origin xyz="0 0 ${chassis_height/2}" rpy="0 0 0"/>
   </joint>
 <!--chassis and cup holder tray-->
 <joint name="chassis_joint" type="fixed">
-    <parent link="chassis"/>
-    <child link="cup_holder_tray"/>
+    <parent link="${robot_name}/chassis"/>
+    <child link="${robot_name}/cup_holder_tray"/>
     <origin xyz="0 0 ${chassis_height/2+standoff_height+tray_height/2}" rpy="0 0 0"/>
 </joint>
 <!--chassis and standoff rods-->
 <joint name="xpyp_standoff_joint" type="fixed">
-    <parent link="chassis"/>
-    <child link="xpyp_standoff"/>
+    <parent link="${robot_name}/chassis"/>
+    <child link="${robot_name}/xpyp_standoff"/>
     <origin xyz="${tray_diameter/4} ${tray_diameter/4} ${chassis_height/2+standoff_height/2}" rpy="0 0 0"/>
 </joint>
 <joint name="xpyn_standoff_joint" type="fixed">
-    <parent link="chassis"/>
-    <child link="xpyn_standoff"/>
+    <parent link="${robot_name}/chassis"/>
+    <child link="${robot_name}/xpyn_standoff"/>
     <origin xyz="${tray_diameter/4} ${-tray_diameter/4} ${chassis_height/2+standoff_height/2}" rpy="0 0 0"/>
 </joint>
 <joint name="xnyp_standoff_joint" type="fixed">
-    <parent link="chassis"/>
-    <child link="xnyp_standoff"/>
+    <parent link="${robot_name}/chassis"/>
+    <child link="${robot_name}/xnyp_standoff"/>
     <origin xyz="${-tray_diameter/4} ${tray_diameter/4} ${chassis_height/2+standoff_height/2}" rpy="0 0 0"/>
 </joint>
 <joint name="xnyn_standoff_joint" type="fixed">
-    <parent link="chassis"/>
-    <child link="xnyn_standoff"/>
+    <parent link="${robot_name}/chassis"/>
+    <child link="${robot_name}/xnyn_standoff"/>
     <origin xyz="${-tray_diameter/4} ${-tray_diameter/4} ${chassis_height/2+standoff_height/2}" rpy="0 0 0"/>
 </joint>
 <!--chassis and wheels-->
 <joint name="left_wheel_joint" type="continuous">
-    <parent link="chassis"/>
-    <child link="left_wheel"/>
+    <parent link="${robot_name}/chassis"/>
+    <child link="${robot_name}/left_wheel"/>
     <origin xyz="0 ${wheel_separation/2} ${-chassis_height/2}" rpy="0 0 0"/>
     <axis xyz="0 1 0" rpy="0 0 0"/>
@@ -119,6 +119,6 @@
 </joint>
 <joint name="right_wheel_joint" type="continuous">
-    <parent link="chassis"/>
-    <child link="right_wheel"/>
+    <parent link="${robot_name}/chassis"/>
+    <child link="${robot_name}/right_wheel"/>
     <origin xyz="0 ${-wheel_separation/2} ${-chassis_height/2}" rpy="0 0 0"/>
     <axis xyz="0 1 0" rpy="0 0 0"/>
@@ -128,6 +128,6 @@
 <!--chassis and casters-->
 <joint name="front_caster_joint" type="continuous">
-    <parent link="chassis"/>
-    <child link="front_caster_wheel_r"/>
+    <parent link="${robot_name}/chassis"/>
+    <child link="${robot_name}/front_caster_wheel_r"/>
     <origin xyz="${chassis_diameter/3} 0 ${-chassis_height/2-wheel_diameter/2+caster_radius}" rpy="0 0 0"/>
     <axis xyz="1 0 0" rpy="0 0 0"/>
@@ -136,6 +136,6 @@
 </joint>
 <joint name="back_caster_joint" type="continuous">
-    <parent link="chassis"/>
-    <child link="back_caster_wheel_r"/>
+    <parent link="${robot_name}/chassis"/>
+    <child link="${robot_name}/back_caster_wheel_r"/>
     <origin xyz="${-chassis_diameter/3} 0 ${-chassis_height/2-wheel_diameter/2+caster_radius}" rpy="0 0 0"/>
     <axis xyz="1 0 0" rpy="0 0 0"/>
@@ -146,6 +146,6 @@
 <xacro:if value="${include_laser}">
     <joint name="laser_joint" type="fixed">
-        <parent link="chassis"/>
-        <child link="laser_scanner"/>
+        <parent link="${robot_name}/chassis"/>
+        <child link="${robot_name}/laser_scanner"/>
         <origin xyz="${chassis_diameter/3} 0 ${chassis_height/2+0.05}" rpy="0 0 0"/>
     </joint>
@@ -163,9 +163,9 @@
         <joint_name>right_wheel_joint</joint_name>
         <joint_name>front_caster_joint</joint_name>
-        <joint_name>front_caster_pitch_joint</joint_name>
-        <joint_name>front_caster_yaw_joint</joint_name>
+        <joint_name>${robot_name}/front_caster_pitch_joint</joint_name>
+        <joint_name>${robot_name}/front_caster_yaw_joint</joint_name>
         <joint_name>back_caster_joint</joint_name>
-        <joint_name>back_caster_pitch_joint</joint_name>
-        <joint_name>back_caster_yaw_joint</joint_name>
+        <joint_name>${robot_name}/back_caster_pitch_joint</joint_name>
+        <joint_name>${robot_name}/back_caster_yaw_joint</joint_name>
     </plugin>
 </gazebo>
@@ -189,10 +189,10 @@
         <publish_odom>true</publish_odom>
         <publish_odom_tf>true</publish_odom_tf>
-        <odometry_frame>odom</odometry_frame>
-        <robot_base_frame>base_link</robot_base_frame>
+        <odometry_frame>${robot_name}/odom</odometry_frame>
+        <robot_base_frame>${robot_name}/base_link</robot_base_frame>
     </plugin>
 </gazebo>
 <!--gazebo materials and frictions coefficients-->
-<gazebo reference="left_wheel">
+<gazebo reference="${robot_name}/left_wheel">
     <kp>1000000000000000000000000000.0</kp>
     <kd>1000000000000000000000000000.0</kd>
@@ -201,5 +201,5 @@
     <material>Gazebo/Black</material>
 </gazebo>
-<gazebo reference="right_wheel">
+<gazebo reference="${robot_name}/right_wheel">
     <kp>1000000000000000000000000000.0</kp>
     <kd>1000000000000000000000000000.0</kd>
@@ -208,5 +208,5 @@
     <material>Gazebo/Black</material>
 </gazebo>
-<gazebo reference="front_caster_wheel_y">
+<gazebo reference="${robot_name}/front_caster_wheel_y">
     <kp>1000000000000000000000000000.0</kp>
     <kd>1000000000000000000000000000.0</kd>
@@ -215,5 +215,5 @@
     <material>Gazebo/Black</material>
 </gazebo>
-<gazebo reference="back_caster_wheel_y">
+<gazebo reference="${robot_name}/back_caster_wheel_y">
     <kp>1000000000000000000000000000.0</kp>
     <kd>1000000000000000000000000000.0</kd>
@@ -222,24 +222,24 @@
     <material>Gazebo/Black</material>
 </gazebo>
-<gazebo reference="chassis">
+<gazebo reference="${robot_name}/chassis">
     <material>${robot_color}</material>
 </gazebo>
-<gazebo reference="cup_holder_tray">
+<gazebo reference="${robot_name}/cup_holder_tray">
     <material>${robot_color}</material>
 </gazebo>
-<gazebo reference="xpyp_standoff">
-    <material>Gazebo/White</material>
-</gazebo>
-<gazebo reference="xpyn_standoff">
-    <material>Gazebo/White</material>
-</gazebo>
-<gazebo reference="xnyp_standoff">
-    <material>Gazebo/White</material>
-</gazebo>
-<gazebo reference="xnyn_standoff">
-    <material>Gazebo/White</material>
-</gazebo>
-<xacro:if value="${include_laser}">
-    <gazebo reference="laser_scanner">
+<gazebo reference="${robot_name}/xpyp_standoff">
+    <material>Gazebo/White</material>
+</gazebo>
+<gazebo reference="${robot_name}/xpyn_standoff">
+    <material>Gazebo/White</material>
+</gazebo>
+<gazebo reference="${robot_name}/xnyp_standoff">
+    <material>Gazebo/White</material>
+</gazebo>
+<gazebo reference="${robot_name}/xnyn_standoff">
+    <material>Gazebo/White</material>
+</gazebo>
+<xacro:if value="${include_laser}">
+    <gazebo reference="${robot_name}/laser_scanner">
         <material>Gazebo/DarkGrey</material>
     </gazebo>
